Commit message: barracuda_description: update URDF and xacro

File: src/barracuda_description/urdf/barracuda.urdf (robot description, URDF)
Before this commit: robot barracuda, 25 links, 24 joints
Joints:
- joint zedm_base_joint: parent barracuda/barracuda_link -> barracuda/base_link

File: src/barracuda_description/urdf/barracuda.xacro (robot description, xacro)
@@ -41,5 +41,5 @@
     <xacro:altimeter parent_link="$(arg namespace)/barracuda_link" altimeter_name="ping1d" namespace="$(arg namespace)" />
     <xacro:include filename="$(find barracuda_description)/urdf/depth_camera.xacro"/>
-    <xacro:depth_camera parent_link="$(arg namespace)/barracuda_link" namespace="$(arg namespace)"/>
+    <xacro:depth_camera parent_link="$(arg namespace)/base_link" namespace="$(arg namespace)"/>
     <gazebo>
         <plugin name="uuv_plugin" filename="libuuv_underwater_object_ros_plugin.so">
